File: hardware/fpga.sch (KiCad schematic (older format))
At the start: 0 parts

Commit message: Finish FTDI schematic, add datasheets
Parts:
- added U? (x9): LFE5U-12F-6BG256C, w_smd_bga:cabga256, symbol Lattice_ECP5_LFE5U-cabga256:LFE5U-12F-6BG256C
Connections:
- new net GND: U?.A1 (GND), U?.A16 (GND), U?.D15 (GND), U?.D2 (GND), U?.F8 (GND), U?.F9 (GND), U?.G10 (GND), U?.G8 (GND), U?.H1 (GND), U?.H10 (GND), U?.H16 (GND), U?.H8 (GND), U?.H9 (GND), U?.J10 (GND), U?.J8 (GND), U?.J9 (GND), U?.K10 (GND), U?.K6 (GND), U?.K7 (GND), U?.K8 (GND), U?.K9 (GND), U?.N15 (GND), U?.N2 (GND), U?.T1 (GND), U?.T12 (GND), U?.T16 (GND), U?.T5 (GND)
- new net TCK: U?.T10 (TCK)
- new net TDI: U?.R11 (TDI)
- new net TDO: U?.M10 (TDO)
- new net TMS: U?.T11 (TMS)
- new net VCC: U?.G6 (VCC), U?.G7 (VCC), U?.G9 (VCC), U?.L10 (VCC), U?.L8 (VCC), U?.L9 (VCC)
- new net VCCAUX: U?.G11 (VCCAUX), U?.L7 (VCCAUX)
