File: hardware/fpga.sch (KiCad schematic (older format))
At the start: 9 parts

Commit message: Add oscilator, flash, ram
Parts:
- added C301: 0.1uF, symbol Device:C_Small
- added D?: Red, symbol Device:LED_Small
- added D?: Green, symbol Device:LED_Small
- added R? (x15): 10k, symbol Device:R_Small
- added R? (x3): 4.7k, symbol Device:R_Small
- added R? (x3): 1k, symbol Device:R_Small
- added R? (x2): 360R, symbol Device:R_Small
- added U?: W25Q32JVSS, Package_SO:SOIC-8_5.275x5.275mm_P1.27mm, symbol Memory_Flash:W25Q32JVSS
- added U? (x2): LY68L6400SLIT, Package_SO:SOIC-8_3.9x4.9mm_P1.27mm, symbol Memory_Flash:W25Q32JVSS
- added X301: 25Mhz, Oscillator:Oscillator_SMD_Abracon_ASE-4Pin_3.2x2.5mm, symbol oscilator:S3D25.000000A20F30T
- gave numbers to parts that had none: 1
Connections:
- net labels added: CLK_25Mhz, FLASH_CLK, FLASH_IO0, FLASH_IO1, FLASH_IO2, FLASH_IO3, FPGA_DONE, FPGA_INITN, RAM0_CLK, RAM0_IO0, RAM0_IO1, RAM0_IO2, RAM0_IO3, RAM1_CLK, RAM1_IO0, RAM1_IO1, RAM1_IO2, RAM1_IO3, ~FLASH_CS~, ~RAM0_CS~, ~RAM1_CS~
- wire segments 74 -> 209
- no-connect marks 0 -> 8
Other:
- moved on the sheet: U301A, U301B, U301C, U301D, U301E, U301F, U301G, U301H

Commit message: More stuff
Parts:
- C301: footprint (none) -> Capacitor_SMD:C_0603_1608Metric
- D301, D302: renamed from D?; footprint (none) -> LED_SMD:LED_0603_1608Metric
- R301, R302, R303, R304, R305, R306, R307, R308, R309, R310, R311, R312, R313, R314, R315, R316, R317, R318, R319, R320, R321, R322, R323: renamed from R?; footprint (none) -> Resistor_SMD:R_0603_1608Metric
- U301: footprint w_smd_bga:cabga256 -> Package_BGA:BGA-256_14.0x14.0mm_Layout16x16_P0.8mm_Ball0.45mm_Pad0.32mm_NSMD
- U302, U304: renamed from U?; footprint Package_SO:SOIC-8_3.9x4.9mm_P1.27mm -> Package_SO:SOIC-8_5.23x5.23mm_P1.27mm
- U303: renamed from U?; footprint Package_SO:SOIC-8_5.275x5.275mm_P1.27mm -> Package_SO:SOIC-8_5.23x5.23mm_P1.27mm
