File: hardware/power.sch (KiCad schematic (older format))
At the start: 16 parts, among them U201 M2406-ADJ, U202 M2406-ADJ, U203 XC6206P25

Commit message: Finish FTDI schematic, add datasheets
Connections:
- net GND: now also U201.1 (EN), U202.1 (EN)
- net VIN: no longer U201.1 (EN), U202.1 (EN)
Changed lines of the file:
@@
 	2800 3700 3100 3700
 Connection ~ 3550 3700
-Wire Wire Line
-	3550 3700 3800 3700
-Wire Wire Line
-	3800 3800 3800 3700
-Connection ~ 3800 3700
-Wire Wire Line
-	3800 3700 4200 3700
 $Comp
 L power:GND #PWR0201
@@
 	6900 3750 6900 3700
 Connection ~ 6900 3700
-Wire Wire Line
-	3800 3800 4200 3800
 $Comp
 L M3406:M2406-ADJ U202
@@
 $EndComp
 Connection ~ 3550 4950
-Wire Wire Line
-	3550 4950 3800 4950
-Wire Wire Line
-	3800 5050 3800 4950
-Connection ~ 3800 4950
-Wire Wire Line
-	3800 4950 4200 4950
 $Comp
 L power:GND #PWR0202
@@
 Connection ~ 5700 4950
 Wire Wire Line
-	3800 5050 4200 5050
-Wire Wire Line
 	5700 4950 5850 4950
 $Comp
@@
 Wire Wire Line
 	3100 3700 3550 3700
+Wire Wire Line
+	3550 4950 4200 4950
+Wire Wire Line
+	3550 3700 4200 3700
+Wire Wire Line
+	4200 5050 3900 5050
+Wire Wire Line
+	3900 5050 3900 5750
+Wire Wire Line
+	3900 5750 1850 5750
+Wire Wire Line
+	4200 3800 4150 3800
+Wire Wire Line
+	4150 3800 4150 4350
+Wire Wire Line
+	4150 4350 1850 4350
+Wire Wire Line
+	1850 4350 1850 5750
+Connection ~ 1850 4350
+Text HLabel 1450 4350 0    50   Input ~ 0
+ENABLE
+Wire Wire Line
+	1450 4350 1600 4350
+$Comp
+L power:GND #PWR?
+U 1 1 5F2149D1
+P 1600 4600
+F 0 "#PWR?" H 1600 4350 50  0001 C CNN
+F 1 "GND" H 1605 4427 50  0000 C CNN
+F 2 "" H 1600 4600 50  0001 C CNN
+F 3 "" H 1600 4600 50  0001 C CNN
+	1    1600 4600
+	1    0    0    -1
+$EndComp
+Wire Wire Line
+	1600 4350 1600 4600
+Connection ~ 1600 4350
+Wire Wire Line
+	1600 4350 1850 4350
 $EndSCHEMATC

Commit message: More stuff
Parts:
- C201, C202, C203, C204, C205, C206, C207: footprint (none) -> Capacitor_SMD:C_0603_1608Metric
- R201, R202, R203, R204: footprint (none) -> Resistor_SMD:R_0603_1608Metric
Changed lines of the file:
@@
 F 0 "R203" V 4954 3800 50  0000 C CNN
 F 1 "6.8k" V 5045 3800 50  0000 C CNN
-F 2 "" H 5150 3800 50  0001 C CNN
+F 2 "Resistor_SMD:R_0603_1608Metric" H 5150 3800 50  0001 C CNN
 F 3 "~" H 5150 3800 50  0001 C CNN
 	1    5150 3800
@@
 F 0 "R201" H 4891 4054 50  0000 R CNN
 F 1 "1.5k" H 4891 4145 50  0000 R CNN
-F 2 "" H 4950 4100 50  0001 C CNN
+F 2 "Resistor_SMD:R_0603_1608Metric" H 4950 4100 50  0001 C CNN
 F 3 "~" H 4950 4100 50  0001 C CNN
 	1    4950 4100
@@
 F 0 "C201" H 3642 3846 50  0000 L CNN
 F 1 "10uF" H 3642 3755 50  0000 L CNN
-F 2 "" H 3550 3800 50  0001 C CNN
+F 2 "Capacitor_SMD:C_0603_1608Metric" H 3550 3800 50  0001 C CNN
 F 3 "~" H 3550 3800 50  0001 C CNN
 	1    3550 3800
@@
 F 0 "C205" H 5792 3946 50  0000 L CNN
 F 1 "10uF" H 5792 3855 50  0000 L CNN
-F 2 "" H 5700 3900 50  0001 C CNN
+F 2 "Capacitor_SMD:C_0603_1608Metric" H 5700 3900 50  0001 C CNN
 F 3 "~" H 5700 3900 50  0001 C CNN
 	1    5700 3900
@@
 F 0 "C203" V 5071 3900 50  0000 C CNN
 F 1 "22pF" V 5162 3900 50  0000 C CNN
-F 2 "" H 5300 3900 50  0001 C CNN
+F 2 "Capacitor_SMD:C_0603_1608Metric" H 5300 3900 50  0001 C CNN
 F 3 "~" H 5300 3900 50  0001 C CNN
 	1    5300 3900
@@
 F 0 "C207" H 6992 3896 50  0000 L CNN
 F 1 "1uF" H 6992 3805 50  0000 L CNN
-F 2 "" H 6900 3850 50  0001 C CNN
+F 2 "Capacitor_SMD:C_0603_1608Metric" H 6900 3850 50  0001 C CNN
 F 3 "~" H 6900 3850 50  0001 C CNN
 	1    6900 3850
@@
 F 0 "R204" V 4954 5050 50  0000 C CNN
 F 1 "100k" V 5045 5050 50  0000 C CNN
-F 2 "" H 5150 5050 50  0001 C CNN
+F 2 "Resistor_SMD:R_0603_1608Metric" H 5150 5050 50  0001 C CNN
 F 3 "~" H 5150 5050 50  0001 C CNN
 	1    5150 5050
@@
 F 0 "R202" H 4891 5304 50  0000 R CNN
 F 1 "120k" H 4891 5395 50  0000 R CNN
-F 2 "" H 4950 5350 50  0001 C CNN
+F 2 "Resistor_SMD:R_0603_1608Metric" H 4950 5350 50  0001 C CNN
 F 3 "~" H 4950 5350 50  0001 C CNN
 	1    4950 5350
@@
 F 0 "C202" H 3642 5096 50  0000 L CNN
 F 1 "10uF" H 3642 5005 50  0000 L CNN
-F 2 "" H 3550 5050 50  0001 C CNN
+F 2 "Capacitor_SMD:C_0603_1608Metric" H 3550 5050 50  0001 C CNN
 F 3 "~" H 3550 5050 50  0001 C CNN
 	1    3550 5050
@@
 F 0 "C206" H 5792 5196 50  0000 L CNN
 F 1 "10uF" H 5792 5105 50  0000 L CNN
-F 2 "" H 5700 5150 50  0001 C CNN
+F 2 "Capacitor_SMD:C_0603_1608Metric" H 5700 5150 50  0001 C CNN
 F 3 "~" H 5700 5150 50  0001 C CNN
 	1    5700 5150
@@
 F 0 "C204" V 5071 5150 50  0000 C CNN
 F 1 "22pF" V 5162 5150 50  0000 C CNN
-F 2 "" H 5300 5150 50  0001 C CNN
+F 2 "Capacitor_SMD:C_0603_1608Metric" H 5300 5150 50  0001 C CNN
 F 3 "~" H 5300 5150 50  0001 C CNN
 	1    5300 5150
